File: pcb/foxbadge/foxbadge.kicad_pcb (KiCad board)
At the start: 2 copper layers, 79.3 x 73.4 mm, 23 parts, among them J1 Display_Connector, J2 Bat_n, J3 Bat_p, SW1 SW_Push_45deg, SW2 SW_Push_45deg, SW3 SW_Push_45deg, SW4 SW_Push_45deg, SW5 SW_Slide_DPDT, U1 XIAO-ESP32-C6-SMD

Commit message: Pictures and Updates
Other:
- board text added: "Mark Scharonow"
Changed lines of the file:
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@@
 		(layer "Edge.Cuts")
+	)
+	(gr_text "Mark Scharonow"
+		(at 106.18 59.19 0)
+		(layer "F.SilkS")
+		(effects
+			(font
+				(size 1.5 1.5)
+				(thickness 0.3)
+				(bold yes)
+			)
+			(justify left bottom)
+		)
 	)
 	(segment
